File: PowerDistributorV2.kicad_sch (KiCad schematic)
At the start: 21 parts, among them J1 F1, J10 D2, J11 D3, J12 D4, J13 D5, J14 D6, J15 D7, J16 D8, J17 PWR, J2 F2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

Commit message: change power connector, add markings, logos and measurements
Parts:
- J17: footprint GSI_footprints:Wago-250-502 -> GSI_footprints:Wago-745-102
Changed lines of the file:
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@@
   (junction (at 88.9 72.39) (diameter 0) (color 0 0 0 0)
   )
-  (junction (at 104.14 50.8) (diameter 0) (color 0 0 0 0)
-  )
   (junction (at 110.49 163.83) (diameter 0) (color 0 0 0 0)
   )
@@
     (stroke (width 0) (type default))
   )
-  (wire (pts (xy 104.14 50.8) (xy 110.49 50.8))
+  (wire (pts (xy 101.6 50.8) (xy 110.49 50.8))
     (stroke (width 0) (type default))
   )
@@
     (stroke (width 0) (type default))
   )
-  (wire (pts (xy 101.6 50.8) (xy 104.14 50.8))
-    (stroke (width 0) (type default))
-  )
   (wire (pts (xy 83.82 72.39) (xy 88.9 72.39))
     (stroke (width 0) (type default))
@@
       (effects (font (size 1.27 1.27)))
     )
-    (property "Footprint" "GSI_footprints:Wago-250-502" (at 101.6 45.72 0)
-      (effects (font (size 1.27 1.27)) hide)
-    )
-    (property "Datasheet" "~" (at 101.6 45.72 0)
-      (effects (font (size 1.27 1.27)) hide)
-    )
+    (property "Footprint" "GSI_footprints:Wago-745-102" (at 101.6 45.72 0)
+      (effects (font (size 1.27 1.27)) hide)
+    )
+    (property "Datasheet" "https://www.wago.com/global/pcb-terminal-blocks-and-pluggable-connectors/terminal-strip-with-jumper-slot/p/745-102" (at 101.6 45.72 0)
+      (effects (font (size 1.27 1.27)) hide)
+    )
